File: carte pami/carte pami.kicad_pcb (KiCad board)
At the start: 2 copper layers, 60.3 x 76.8 mm, 16 parts, among them J1 RJ25, J2 Battery 6,4V, J3 ARU, J4 RJ25, J5 Conn_01x06_Pin, J6 Conn_01x19_Pin, J7 Conn_01x19_Pin, SW2 SW_Push_DPDT, U1 ESP32_NODEMCU, U2 7805

Commit message: updates
Routing:
- net GND: track 114.5 -> 139.8 mm
- net G21: track 42.5 -> 30.1 mm
- net TXD1: track 34.0 -> 32.4 mm, vias 1 -> 0
- net RXD1: track 24.1 -> 23.1 mm, vias 1 -> 0
Changed lines of the file:
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@@
       (disableapertmacros false)
       (usegerberextensions true)
-      (usegerberattributes true)
-      (usegerberadvancedattributes true)
+      (usegerberattributes false)
+      (usegerberadvancedattributes false)
       (creategerberjobfile false)
       (dashed_line_dash_ratio 12.000000)
@@
       (psa4output false)
       (plotreference true)
-      (plotvalue false)
+      (plotvalue true)
       (plotinvisibletext false)
       (sketchpadsonfab false)
@@
   (segment (start 150 57.75) (end 150 53) (width 1.5) (layer "B.Cu") (net 5))
   (segment (start 110.49 99.06) (end 116.84 105.41) (width 1.5) (layer "B.Cu") (net 5))
+  (segment (start 144.535 93.035) (end 145.415 93.035) (width 1.5) (layer "B.Cu") (net 5))
+  (segment (start 142.25 72.5) (end 142.25 90.75) (width 1.5) (layer "B.Cu") (net 5))
   (segment (start 141.29 63.46) (end 141.29 63.5) (width 1.5) (layer "B.Cu") (net 5))
   (segment (start 141.29 63.46) (end 141.29 66.04) (width 1.5) (layer "B.Cu") (net 5))
-  (segment (start 144.47 93.035) (end 145.415 93.035) (width 1.5) (layer "B.Cu") (net 5))
   (segment (start 143.5 61.25) (end 141.29 63.46) (width 1.5) (layer "B.Cu") (net 5))
   (segment (start 100.965 99.06) (end 104.475 99.06) (width 1.5) (layer "B.Cu") (net 5))
@@
   (segment (start 145 69.75) (end 141.29 66.04) (width 1.5) (layer "B.Cu") (net 5))
   (segment (start 99.695 83.82) (end 98.425 85.09) (width 1.5) (layer "B.Cu") (net 5))
+  (segment (start 142.25 90.75) (end 144.535 93.035) (width 1.5) (layer "B.Cu") (net 5))
+  (segment (start 145 69.75) (end 142.25 72.5) (width 1.5) (layer "B.Cu") (net 5))
   (segment (start 133.985 66.04) (end 130.475 66.04) (width 1.5) (layer "B.Cu") (net 5))
   (segment (start 146.5 61.25) (end 150 57.75) (width 1.5) (layer "B.Cu") (net 5))
@@
   (segment (start 100.965 83.82) (end 104.475 83.82) (width 1.5) (layer "B.Cu") (net 5))
   (segment (start 145.445 61.25) (end 146.5 61.25) (width 1.5) (layer "B.Cu") (net 5))
-  (segment (start 119.75 110.75) (end 122 110.75) (width 0.5) (layer "B.Cu") (net 6))
-  (segment (start 119.375 106.68) (end 119.375 110.375) (width 0.5) (layer "B.Cu") (net 6))
-  (segment (start 123 104.885) (end 104.475 86.36) (width 0.5) (layer "B.Cu") (net 6))
-  (segment (start 122 110.75) (end 123 109.75) (width 0.5) (layer "B.Cu") (net 6))
+  (segment (start 104.475 86.475) (end 119.5 101.5) (width 0.5) (layer "F.Cu") (net 6))
+  (segment (start 119.5 106.555) (end 119.375 106.68) (width 0.5) (layer "F.Cu") (net 6))
+  (segment (start 104.475 86.36) (end 104.475 86.475) (width 0.5) (layer "F.Cu") (net 6))
+  (segment (start 119.5 101.5) (end 119.5 106.555) (width 0.5) (layer "F.Cu") (net 6))
   (segment (start 104.475 86.36) (end 100.965 86.36) (width 0.5) (layer "B.Cu") (net 6))
-  (segment (start 119.375 110.375) (end 119.75 110.75) (width 0.5) (layer "B.Cu") (net 6))
-  (segment (start 123 109.75) (end 123 104.885) (width 0.5) (layer "B.Cu") (net 6))
   (segment (start 121.285 108.58) (end 121.285 106.045) (width 0.5) (layer "B.Cu") (net 7))
   (segment (start 121.285 106.045) (end 109.22 93.98) (width 0.5) (layer "B.Cu") (net 7))
@@
   (segment (start 104.475 78.74) (end 100.965 78.74) (width 0.5) (layer "B.Cu") (net 25))
   (segment (start 100.965 81.28) (end 104.475 81.28) (width 0.5) (layer "B.Cu") (net 26))
-  (segment (start 106.75 90.75) (end 106.75 104.62) (width 0.5) (layer "F.Cu") (net 27))
-  (segment (start 106.75 104.62) (end 104.18 107.19) (width 0.5) (layer "F.Cu") (net 27))
-  (segment (start 106.5 90.5) (end 106.75 90.75) (width 0.5) (layer "F.Cu") (net 27))
-  (via (at 106.5 90.5) (size 1.2) (drill 0.6) (layers "F.Cu" "B.Cu") (net 27))
-  (segment (start 104.475 88.9) (end 106.075 90.5) (width 0.5) (layer "B.Cu") (net 27))
+  (segment (start 104.18 107.19) (end 102.75 105.76) (width 0.5) (layer "F.Cu") (net 27))
+  (segment (start 102.75 90.625) (end 104.475 88.9) (width 0.5) (layer "F.Cu") (net 27))
+  (segment (start 102.75 105.76) (end 102.75 90.625) (width 0.5) (layer "F.Cu") (net 27))
   (segment (start 100.965 88.9) (end 104.475 88.9) (width 0.5) (layer "B.Cu") (net 27))
-  (segment (start 106.075 90.5) (end 106.5 90.5) (width 0.5) (layer "B.Cu") (net 27))
   (segment (start 109 112.25) (end 105.94 112.25) (width 0.5) (layer "F.Cu") (net 28))
-  (segment (start 109.75 94) (end 109.75 111.5) (width 0.5) (layer "F.Cu") (net 28))
+  (segment (start 109.75 96.75) (end 109.75 111.5) (width 0.5) (layer "F.Cu") (net 28))
   (segment (start 109.75 111.5) (end 109 112.25) (width 0.5) (layer "F.Cu") (net 28))
+  (segment (start 104.475 91.44) (end 104.475 91.475) (width 0.5) (layer "F.Cu") (net 28))
   (segment (start 105.94 112.25) (end 104.18 110.49) (width 0.5) (layer "F.Cu") (net 28))
-  (segment (start 108 92.25) (end 109.75 94) (width 0.5) (layer "F.Cu") (net 28))
-  (via (at 108 92.25) (size 1.2) (drill 0.6) (layers "F.Cu" "B.Cu") (net 28))
-  (segment (start 108 92.25) (end 105.25 92.25) (width 0.5) (layer "B.Cu") (net 28))
+  (segment (start 104.475 91.475) (end 109.75 96.75) (width 0.5) (layer "F.Cu") (net 28))
   (segment (start 104.475 91.44) (end 100.965 91.44) (width 0.5) (layer "B.Cu") (net 28))
   (segment (start 104.475 91.475) (end 104.475 91.44) (width 0.5) (layer "B.Cu") (net 28))
-  (segment (start 105.25 92.25) (end 104.475 91.475) (width 0.5) (layer "B.Cu") (net 28))
   (segment (start 104.475 96.52) (end 100.965 96.52) (width 0.5) (layer "B.Cu") (net 29))
   (segment (start 130.475 99.06) (end 133.985 99.06) (width 1) (layer "B.Cu") (net 30))

Commit message: Carte elec
Parts:
- removed H4: MountingHole, MountingHole:MountingHole_3.2mm_M3_Pad
- removed J7: Conn_01x19_Pin, Connector_PinHeader_2.54mm:PinHeader_1x19_P2.54mm_Vertical
- removed SW2: SW_Push_DPDT, Button_Switch_THT:SW_CuK_JS202011CQN_DPDT_Straight
- H1, H2, H3: footprint MountingHole:MountingHole_3.2mm_M3_Pad -> MountingHole:MountingHole_3.2mm_M3
- J1: value RJ25 -> RJ25_Driver
- J2, J3: footprint Carte PAMI:Connecteur Batterie,... -> Connector_JST:JST_XH_B2B-XH-A_1x02_P2.50mm_Vertical
- J4: value RJ25 -> Conn_SR04; footprint Carte PAMI:Rj25 -> Connector_JST:JST_PH_B4B-PH-K_1x04_P2.00mm_Vertical
- J5: value Conn_01x06_Pin -> Conn_Jack; footprint Connector_PinHeader_2.54mm:PinHeader_1x06_P2.54mm_Vertical -> Connector_JST:JST_PH_B2B-PH-K_1x02_P2.00mm_Vertical
- J6: value Conn_01x19_Pin -> Conn_Servo; footprint Connector_PinHeader_2.54mm:PinHeader_1x19_P2.54mm_Vertical -> Connector_JST:JST_PH_B3B-PH-K_1x03_P2.00mm_Vertical
- U2: value 7805 -> LM7805_TO220
- moved J5 51.6 mm to (137.0, 52.8)
- moved J1 46.0 mm to (120.9, 63.4), turned to 90 degrees
- moved C1 38.9 mm to (124.1, 98.8)
- moved C2 38.6 mm to (124.2, 81.8)
- moved H2 37.8 mm to (124.8, 74.0)
- moved J4 37.7 mm to (137.0, 72.5)
- moved J6 37.2 mm to (137.2, 61.8), turned to -90 degrees
- moved U2 36.0 mm to (124.2, 92.8)
- moved H3 19.6 mm to (109.8, 100.0)
- moved H1 13.6 mm to (109.8, 52.8)
- moved J3 13.0 mm to (137.0, 86.0)
- moved J2 11.4 mm to (137.0, 97.2)
Connections:
- J1 pad 1: G22 -> SCL
- J1 pad 2: G21 -> SDA
- J4 pad 1: Net-(J5-Pin_1) -> 5v
- J4 pad 2: Net-(J5-Pin_2) -> Trigger
- J4 pad 3: Net-(J5-Pin_3) -> Echo
- J4 pad 4: Net-(J5-Pin_4) -> GND
- J5 pad 1: Net-(J5-Pin_1) -> 3v3
- J5 pad 2: Net-(J5-Pin_2) -> Jack
- J6 pad 1: CLK -> GND
- J6 pad 2: SD0 -> 5v
- J6 pad 3: SD1 -> PWM_Servo
- U1 pad J4_10: G5 -> Trigger
- U1 pad J4_11: G17 -> unconnected-(U1-G17-PadJ4_11)
- U1 pad J4_12: G16 -> unconnected-(U1-G16-PadJ4_12)
- U1 pad J4_13: G4 -> unconnected-(U1-G4-PadJ4_13)
- U1 pad J4_14: G0 -> unconnected-(U1-G0-PadJ4_14)
- U1 pad J4_15: G2 -> unconnected-(U1-G2-PadJ4_15)
- U1 pad J4_16: G15 -> unconnected-(U1-G15-PadJ4_16)
- U1 pad J4_17: SD1 -> unconnected-(U1-SD1-PadJ4_17)
- U1 pad J4_18: SD0 -> unconnected-(U1-SD0-PadJ4_18)
- U1 pad J4_19: CLK -> unconnected-(U1-CLK-PadJ4_19)
- U1 pad J4_2: G23 -> unconnected-(U1-G23-PadJ4_2)
- U1 pad J4_3: G22 -> SCL
- U1 pad J4_4: TXD1 -> unconnected-(U1-TXD-PadJ4_4)
- U1 pad J4_5: RXD1 -> unconnected-(U1-RXD-PadJ4_5)
- U1 pad J4_6: G21 -> SDA
- U1 pad J4_8: G19 -> Jack
- U1 pad J4_9: G18 -> Echo
- U1 pad J5_10: G26 -> unconnected-(U1-G26-PadJ5_10)
- U1 pad J5_11: G25 -> unconnected-(U1-G25-PadJ5_11)
- U1 pad J5_12: G33 -> unconnected-(U1-G33-PadJ5_12)
- U1 pad J5_13: G32 -> unconnected-(U1-G32-PadJ5_13)
- U1 pad J5_14: G35 -> unconnected-(U1-G35-PadJ5_14)
- U1 pad J5_15: G34 -> unconnected-(U1-G34-PadJ5_15)
- U1 pad J5_16: SM -> unconnected-(U1-SN-PadJ5_16)
- U1 pad J5_17: SP -> unconnected-(U1-SP-PadJ5_17)
- U1 pad J5_18: EN -> unconnected-(U1-EN-PadJ5_18)
- U1 pad J5_2: CMD -> unconnected-(U1-CMD-PadJ5_2)
- U1 pad J5_3: SD3 -> unconnected-(U1-SD3-PadJ5_3)
- U1 pad J5_4: SD2 -> unconnected-(U1-SD2-PadJ5_4)
- U1 pad J5_5: G13 -> unconnected-(U1-G13-PadJ5_5)
- U1 pad J5_7: G12 -> unconnected-(U1-G12-PadJ5_7)
- U1 pad J5_8: G14 -> unconnected-(U1-G14-PadJ5_8)
- U1 pad J5_9: G27 -> PWM_Servo
Routing:
- net GND: track 139.8 -> 0.00 mm
- net V-M: track 97.0 -> 0.00 mm
- net TXD1: track 32.4 -> 0.00 mm
- net G21: track 30.1 -> 0.00 mm
- net G22: track 28.8 -> 0.00 mm
- net RXD1: track 23.1 -> 0.00 mm
- net 5v: track 22.9 -> 0.00 mm
- net RXD: track 19.6 -> 0.00 mm
- net TXD: track 14.7 -> 0.00 mm
- net Net-(J2-Pin_1): track 10.0 -> 0.00 mm
- net Net-(J5-Pin_1): track 8.29 -> 0.00 mm
- net Net-(J5-Pin_5): track 7.76 -> 0.00 mm
- net Net-(J5-Pin_3): track 7.24 -> 0.00 mm
- net Net-(J5-Pin_6): track 5.75 -> 0.00 mm
- net Net-(J5-Pin_2): track 5.23 -> 0.00 mm
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Other:
- board text removed: "Conn bonus"
- board text removed: "ON|OFF"
- board text removed: "Serial driver"
