File: carte pami/carte pami.kicad_sch (KiCad schematic)
At the start: 16 parts, among them J1 RJ25, J2 Battery 6,4V, J3 ARU, J4 RJ25, J5 Conn_01x06_Pin, J6 Conn_01x19_Pin, J7 Conn_01x19_Pin, SW2 SW_Push_DPDT, U1 ESP32_NODEMCU, U2 LM7805_TO220

Commit message: Carte elec
Parts:
- removed H4: MountingHole, MountingHole:MountingHole_3.2mm_M3_Pad, symbol Mechanical:MountingHole
- removed J4: RJ25, Carte PAMI:Rj25, symbol Connector:RJ25
- removed J5: Conn_01x06_Pin, Connector_PinHeader_2.54mm:PinHeader_1x06_P2.54mm_Vertical, symbol Connector:Conn_01x06_Pin
- removed J6, J7: Conn_01x19_Pin, Connector_PinHeader_2.54mm:PinHeader_1x19_P2.54mm_Vertical, symbol Connector:Conn_01x19_Pin
- removed SW2: SW_Push_DPDT, Button_Switch_THT:SW_CuK_JS202011CQN_DPDT_Straight, symbol Switch:SW_Push_DPDT
- added J4: Conn_SR04, Connector_JST:JST_PH_B4B-PH-K_1x04_P2.00mm_Vertical, symbol Connector:Conn_01x04_Pin
- added J5: Conn_Jack, Connector_JST:JST_PH_B2B-PH-K_1x02_P2.00mm_Vertical, symbol Connector:Conn_01x02_Pin
- added J6: Conn_Servo, Connector_JST:JST_PH_B3B-PH-K_1x03_P2.00mm_Vertical, symbol Connector:Conn_01x03_Pin
- H1, H2, H3: footprint MountingHole:MountingHole_3.2mm_M3_Pad -> MountingHole:MountingHole_3.2mm_M3
- J1: value RJ25 -> RJ25_Driver
- J2, J3: footprint Carte PAMI:Connecteur Batterie,... -> Connector_JST:JST_XH_B2B-XH-A_1x02_P2.50mm_Vertical
Connections:
- net 3v3: now also J5.1 (Pin_1)
- net 5v: now also J4.1 (Pin_1), J6.2 (Pin_2)
- net GND: now also J4.4 (Pin_4), J6.1 (Pin_1)
- net CLK: no longer names the net of U1.J4_19 (CLK)
- net CMD: no longer names the net of U1.J5_2 (CMD)
- net EN: no longer names the net of U1.J5_18 (EN)
- net G0: no longer names the net of U1.J4_14 (G0)
- net G12: no longer names the net of U1.J5_7 (G12)
- net G13: no longer names the net of U1.J5_5 (G13)
- net G14: no longer names the net of U1.J5_8 (G14)
- net G15: no longer names the net of U1.J4_16 (G15)
- net G16: no longer names the net of U1.J4_12 (G16)
- net G17: no longer names the net of U1.J4_11 (G17)
- net G18 renamed Echo
- net Echo: now also J4.3 (Pin_3)
- net G19 renamed Jack
- net Jack: now also J5.2 (Pin_2)
- net G2: no longer names the net of U1.J4_15 (G2)
- net G21 renamed SDA
- net G22 renamed SCL
- net G23: no longer names the net of U1.J4_2 (G23)
- net G25: no longer names the net of U1.J5_11 (G25)
- net G26: no longer names the net of U1.J5_10 (G26)
- net G27 renamed PWM_Servo
- net PWM_Servo: now also J6.3 (Pin_3)
- net G32: no longer names the net of U1.J5_13 (G32)
- net G33: no longer names the net of U1.J5_12 (G33)
- net G34: no longer names the net of U1.J5_15 (G34)
- net G35: no longer names the net of U1.J5_14 (G35)
- net G4: no longer names the net of U1.J4_13 (G4)
- net G5 renamed Trigger
- net Trigger: now also J4.2 (Pin_2)
- net RXD1: no longer names the net of U1.J4_5 (RXD)
- net SD0: no longer names the net of U1.J4_18 (SD0)
- net SD1: no longer names the net of U1.J4_17 (SD1)
- net SD2: no longer names the net of U1.J5_4 (SD2)
- net SD3: no longer names the net of U1.J5_3 (SD3)
- net SM: no longer names the net of U1.J5_16 (SN)
- net SP: no longer names the net of U1.J5_17 (SP)
- net TXD1: no longer names the net of U1.J4_4 (TXD)
- no-connect marks 2 -> 27
